File: Python480.sch (KiCad schematic (older format))
At the start: 29 parts, among them U1 NOIP1SN0480A, U2 LM321, U3 NCP163AMX330TBG, X1 SG-210STF

Commit message: sync
Parts:
- C1, C10, C11, C12, C13, C14, C15, C16, C17, C18, C19, C2, C20, C21, C3, C4, C5, C6, C7, C8, C9: symbol Capacitor:GRM033R61A104ME15D -> Python480-rescue:GRM033R61A104ME15D-Capacitor
- L1, L2: symbol BLM18AG601SN1D:BLM18AG601SN1D -> Python480-rescue:BLM18AG601SN1D-BLM18AG601SN1D
- R1: symbol Resistor:ERJ-1GEF1022C -> Python480-rescue:ERJ-1GEF1022C-Resistor
- U1: symbol Image_Sensor:NOIP1SN0480A -> Python480-rescue:NOIP1SN0480A-Image_Sensor
- U3: symbol doragasu:MCP1711 -> Python480-rescue:MCP1711-doragasu
Changed lines of the file:
@@
 $EndDescr
 $Comp
-L Image_Sensor:NOIP1SN0480A U1
+L Python480-rescue:NOIP1SN0480A-Image_Sensor U1
 U 1 1 602C5332
 P 2450 3400
@@
 	1150 4950 1150 5050
 $Comp
-L Resistor:ERJ-1GEF1022C R1
+L Python480-rescue:ERJ-1GEF1022C-Resistor R1
 U 1 1 602DBEFE
 P 1150 5150
@@
 	500  500  500  5950
 $Comp
-L Capacitor:GRM033R61A104ME15D C4
+L Python480-rescue:GRM033R61A104ME15D-Capacitor C4
 U 1 1 604EA7B5
 P 5800 2300
@@
 	4950 1400 5400 1400
 $Comp
-L Capacitor:GRM033R61A104ME15D C1
+L Python480-rescue:GRM033R61A104ME15D-Capacitor C1
 U 1 1 604EB512
 P 4950 1500
@@
 Connection ~ 4950 1400
 $Comp
-L Capacitor:GRM033R61A104ME15D C2
+L Python480-rescue:GRM033R61A104ME15D-Capacitor C2
 U 1 1 604EBB1C
 P 5400 1500
@@
 	4950 1600 5400 1600
 $Comp
-L Capacitor:GRM033R61A104ME15D C3
+L Python480-rescue:GRM033R61A104ME15D-Capacitor C3
 U 1 1 604EC155
 P 5800 1500
@@
 	5800 1400 6250 1400
 $Comp
-L Capacitor:GRM033R61A104ME15D C6
+L Python480-rescue:GRM033R61A104ME15D-Capacitor C6
 U 1 1 604EC74B
 P 6250 1500
@@
 	6250 1400 6700 1400
 $Comp
-L Capacitor:GRM033R61A104ME15D C9
+L Python480-rescue:GRM033R61A104ME15D-Capacitor C9
 U 1 1 604ECC60
 P 6700 1500
@@
 	6700 1400 7200 1400
 $Comp
-L Capacitor:GRM033R61A104ME15D C12
+L Python480-rescue:GRM033R61A104ME15D-Capacitor C12
 U 1 1 604ED0F8
 P 7200 1500
@@
 	5800 2400 6250 2400
 $Comp
-L Capacitor:GRM033R61A104ME15D C7
+L Python480-rescue:GRM033R61A104ME15D-Capacitor C7
 U 1 1 604F44F5
 P 6250 2300
@@
 	6250 2200 6700 2200
 $Comp
-L Capacitor:GRM033R61A104ME15D C10
+L Python480-rescue:GRM033R61A104ME15D-Capacitor C10
 U 1 1 604F4CAD
 P 6700 2300
@@
 	5800 3050 6300 3050
 $Comp
-L Capacitor:GRM033R61A104ME15D C13
+L Python480-rescue:GRM033R61A104ME15D-Capacitor C13
 U 1 1 604F5246
 P 7200 2300
@@
 $EndComp
 $Comp
-L Capacitor:GRM033R61A104ME15D C14
+L Python480-rescue:GRM033R61A104ME15D-Capacitor C14
 U 1 1 6050232E
 P 7200 2950
@@
 $EndComp
 $Comp
-L Capacitor:GRM033R61A104ME15D C11
+L Python480-rescue:GRM033R61A104ME15D-Capacitor C11
 U 1 1 60502D44
 P 6750 2950
@@
 	6750 2850 7200 2850
 $Comp
-L Capacitor:GRM033R61A104ME15D C8
+L Python480-rescue:GRM033R61A104ME15D-Capacitor C8
 U 1 1 60503308
 P 6300 2950
@@
 	6300 2850 6750 2850
 $Comp
-L Capacitor:GRM033R61A104ME15D C5
+L Python480-rescue:GRM033R61A104ME15D-Capacitor C5
 U 1 1 60503B0B
 P 5800 2950
@@
 Connection ~ 7200 3050
 $Comp
-L Capacitor:GRM033R61A104ME15D C17
+L Python480-rescue:GRM033R61A104ME15D-Capacitor C17
 U 1 1 6050C6C7
 P 7200 3650
@@
 	4700 4800 5000 4800
 $Comp
-L Capacitor:GRM033R61A104ME15D C16
+L Python480-rescue:GRM033R61A104ME15D-Capacitor C16
 U 1 1 6050D4A6
 P 6000 4250
@@
 $EndComp
 $Comp
-L Capacitor:GRM033R61A104ME15D C15
+L Python480-rescue:GRM033R61A104ME15D-Capacitor C15
 U 1 1 6050DE3C
 P 5000 4900
@@
 	5650 2200 5800 2200
 $Comp
-L Capacitor:GRM033R61A104ME15D C18
+L Python480-rescue:GRM033R61A104ME15D-Capacitor C18
 U 1 1 60510477
 P 7450 5000
@@
 	6850 4900 7450 4900
 $Comp
-L BLM18AG601SN1D:BLM18AG601SN1D L2
+L Python480-rescue:BLM18AG601SN1D-BLM18AG601SN1D L2
 U 1 1 603EC076
 P 6250 4900
@@
 $EndComp
 $Comp
-L BLM18AG601SN1D:BLM18AG601SN1D L1
+L Python480-rescue:BLM18AG601SN1D-BLM18AG601SN1D L1
 U 1 1 603FF823
 P 5050 2200
@@
 $EndComp
 $Comp
-L Capacitor:GRM033R61A104ME15D C19
+L Python480-rescue:GRM033R61A104ME15D-Capacitor C19
 U 1 1 603B3C8E
 P 10300 1050
@@
 	8000 2400 8000 4100
 $Comp
-L Capacitor:GRM033R61A104ME15D C20
+L Python480-rescue:GRM033R61A104ME15D-Capacitor C20
 U 1 1 6043665D
 P 8450 3350
@@
 $EndComp
 $Comp
-L Capacitor:GRM033R61A104ME15D C21
+L Python480-rescue:GRM033R61A104ME15D-Capacitor C21
 U 1 1 60447882
 P 10100 3350
@@
 Connection ~ 10100 3150
 $Comp
-L doragasu:MCP1711 U3
+L Python480-rescue:MCP1711-doragasu U3
 U 1 1 604341DF
 P 9500 3350
