File: FPGA.sch (KiCad schematic (older format))
At the start: 2 parts

Commit message: sync
Parts:
- added U? (x3): 10M50SCE144C8G, 10M50SCE144:QFP50P2200X2200X165-145N, symbol 10M50SCE:10M50SCE144C8G
- U?: symbol FPGA:MAX10-10M08DCU324 -> FPGA-rescue:MAX10-10M08DCU324-FPGA
Changed lines of the file:
@@
 EELAYER 30 0
 EELAYER END
-$Descr A4 11693 8268
+$Descr A3 16535 11693
 encoding utf-8
 Sheet 1 1
@@
 $EndComp
 $Comp
-L FPGA:MAX10-10M08DCU324 U?
+L FPGA-rescue:MAX10-10M08DCU324-FPGA U?
 U 1 1 603A2FBE
 P 4360 5690
@@
 	1    0    0    -1
 $EndComp
+$Comp
+L 10M50SCE:10M50SCE144C8G U?
+U 1 1 607366C8
+P 12600 2200
+F 0 "U?" H 12978 2096 50  0000 L CNN
+F 1 "10M50SCE144C8G" H 12978 2005 50  0000 L CNN
+F 2 "10M50SCE144:QFP50P2200X2200X165-145N" H 12600 2200 50  0001 C CNN
+F 3 "" H 12600 2200 50  0001 C CNN
+	1    12600 2200
+	1    0    0    -1
+$EndComp
+$Comp
+L 10M50SCE:10M50SCE144C8G U?
+U 2 1 6073C5EF
+P 13000 3250
+F 0 "U?" H 13028 2996 50  0000 L CNN
+F 1 "10M50SCE144C8G" H 13028 2905 50  0000 L CNN
+F 2 "10M50SCE144:QFP50P2200X2200X165-145N" H 13000 3250 50  0001 C CNN
+F 3 "" H 13000 3250 50  0001 C CNN
+	2    13000 3250
+	1    0    0    -1
+$EndComp
+$Comp
+L 10M50SCE:10M50SCE144C8G U?
+U 3 1 6073EA8F
+P 12700 4700
+F 0 "U?" H 13028 4596 50  0000 L CNN
+F 1 "10M50SCE144C8G" H 13028 4505 50  0000 L CNN
+F 2 "10M50SCE144:QFP50P2200X2200X165-145N" H 12700 4700 50  0001 C CNN
+F 3 "" H 12700 4700 50  0001 C CNN
+	3    12700 4700
+	1    0    0    -1
+$EndComp

Commit message: sync
Parts:
- removed IC?: 10M50SCE144C8G, QFP50P2200X2200X165-145N, symbol FPGA-rescue:10M50SCE144C8G-10M50SCE144C8G
- removed U?: MAX10-10M08DCU324, Package_BGA:BGA-324_15.0x15.0mm_Layout18x18_P0.8mm_Ball0.5mm_Pad0.4mm_NSMD, symbol FPGA-rescue:MAX10-10M08DCU324-FPGA
- removed U? (x3): 10M50SCE144C8G, 10M50SCE144:QFP50P2200X2200X165-145N, symbol 10M50SCE:10M50SCE144C8G
- added U?: 10M50SCE144C8G, 10M50SCE144:QFP50P2200X2200X165-145N, symbol 10M50SCE:10M50SCE144C8G
Connections:
- net labels added: DOU2, DOUT1, DOUT3, DOUT4, DOUT5, DOUT6, DOUT7, DOUT8, DOUT9
- wire segments 0 -> 9
Changed lines of the file:
@@
 $EndDescr
 $Comp
-L FPGA-rescue:10M50SCE144C8G-10M50SCE144C8G IC?
-U 1 1 6011306D
-P 5300 5600
-F 0 "IC?" H 7450 4150 50  0000 L CNN
-F 1 "10M50SCE144C8G" H 7150 3950 50  0000 L CNN
-F 2 "QFP50P2200X2200X165-145N" H 9350 6600 50  0001 L CNN
-F 3 "https://www.intel.com/content/dam/www/programmable/us/en/pdfs/literature/dp/max-10/10m50sc.pdf" H 9350 6500 50  0001 L CNN
-F 4 "FPGA MAX 10 Family 50000 Cells 55nm Technology 1.2V 144-Pin EQFP EP" H 9350 6400 50  0001 L CNN "Description"
-F 5 "1.65" H 9350 6300 50  0001 L CNN "Height"
-F 6 "Intel" H 9350 6200 50  0001 L CNN "Manufacturer_Name"
-F 7 "10M50SCE144C8G" H 9350 6100 50  0001 L CNN "Manufacturer_Part_Number"
-F 8 "989-10M50SCE144C8G" H 9350 6000 50  0001 L CNN "Mouser Part Number"
-F 9 "https://www.mouser.co.uk/ProductDetail/Intel-Altera/10M50SCE144C8G?qs=G%2FX6g08h60s2ThCT%2Fg69Zw%3D%3D" H 9350 5900 50  0001 L CNN "Mouser Price/Stock"
-F 10 "10M50SCE144C8G" H 9350 5800 50  0001 L CNN "Arrow Part Number"
-F 11 "https://www.arrow.com/en/products/10m50sce144c8g/intel" H 9350 5700 50  0001 L CNN "Arrow Price/Stock"
-	1    5300 5600
-	-1   0    0    1
+L 10M50SCE:10M50SCE144C8G U?
+U 4 1 607B5417
+P 2250 2750
+F 0 "U?" H 1942 3215 50  0000 C CNN
+F 1 "10M50SCE144C8G" H 1942 3124 50  0000 C CNN
+F 2 "10M50SCE144:QFP50P2200X2200X165-145N" H 2250 2750 50  0001 C CNN
+F 3 "" H 2250 2750 50  0001 C CNN
+	4    2250 2750
+	-1   0    0    -1
 $EndComp
-$Comp
-L FPGA-rescue:MAX10-10M08DCU324-FPGA U?
-U 1 1 603A2FBE
-P 4360 5690
-F 0 "U?" H 7035 9355 50  0000 C CNN
-F 1 "MAX10-10M08DCU324" H 7035 9264 50  0000 C CNN
-F 2 "Package_BGA:BGA-324_15.0x15.0mm_Layout18x18_P0.8mm_Ball0.5mm_Pad0.4mm_NSMD" H 7260 9640 50  0001 C CNN
-F 3 "https://www.intel.la/content/dam/www/programmable/us/en/pdfs/literature/pt/max-10-product-table.pdf" H 7060 9440 50  0001 C CNN
-	1    4360 5690
-	1    0    0    -1
-$EndComp
-$Comp
-L 10M50SCE:10M50SCE144C8G U?
-U 1 1 607366C8
-P 12600 2200
-F 0 "U?" H 12978 2096 50  0000 L CNN
-F 1 "10M50SCE144C8G" H 12978 2005 50  0000 L CNN
-F 2 "10M50SCE144:QFP50P2200X2200X165-145N" H 12600 2200 50  0001 C CNN
-F 3 "" H 12600 2200 50  0001 C CNN
-	1    12600 2200
-	1    0    0    -1
-$EndComp
-$Comp
-L 10M50SCE:10M50SCE144C8G U?
-U 2 1 6073C5EF
-P 13000 3250
-F 0 "U?" H 13028 2996 50  0000 L CNN
-F 1 "10M50SCE144C8G" H 13028 2905 50  0000 L CNN
-F 2 "10M50SCE144:QFP50P2200X2200X165-145N" H 13000 3250 50  0001 C CNN
-F 3 "" H 13000 3250 50  0001 C CNN
-	2    13000 3250
-	1    0    0    -1
-$EndComp
-$Comp
-L 10M50SCE:10M50SCE144C8G U?
-U 3 1 6073EA8F
-P 12700 4700
-F 0 "U?" H 13028 4596 50  0000 L CNN
-F 1 "10M50SCE144C8G" H 13028 4505 50  0000 L CNN
-F 2 "10M50SCE144:QFP50P2200X2200X165-145N" H 12700 4700 50  0001 C CNN
-F 3 "" H 12700 4700 50  0001 C CNN
-	3    12700 4700
-	1    0    0    -1
-$EndComp
+Wire Wire Line
+	2950 2550 3400 2550
+Wire Wire Line
+	2950 2650 3400 2650
+Wire Wire Line
+	2950 2750 3400 2750
+Wire Wire Line
+	2950 2850 3400 2850
+Wire Wire Line
+	2950 2950 3400 2950
+Wire Wire Line
+	2950 3050 3400 3050
+Wire Wire Line
+	2950 3150 3400 3150
+Wire Wire Line
+	2950 3250 3400 3250
+Wire Wire Line
+	2950 3350 3400 3350
+Text Label 3050 2550 0    50   ~ 0
+DOUT1
+Text Label 3050 2650 0    50   ~ 0
+DOU2
+Text Label 3050 2750 0    50   ~ 0
+DOUT3
+Text Label 3050 2850 0    50   ~ 0
+DOUT4
+Text Label 3050 2950 0    50   ~ 0
+DOUT5
+Text Label 3050 3050 0    50   ~ 0
+DOUT6
+Text Label 3050 3150 0    50   ~ 0
+DOUT7
+Text Label 3050 3250 0    50   ~ 0
+DOUT8
+Text Label 3050 3350 0    50   ~ 0
+DOUT9
 $EndSCHEMATC

Commit message: sync
Parts:
- gave numbers to parts that had none: 1
Other:
- moved on the sheet: U1D
Changed lines of the file:
@@
 $EndDescr
 $Comp
-L 10M50SCE:10M50SCE144C8G U?
+L 10M50SCE:10M50SCE144C8G U1
 U 4 1 607B5417
-P 2250 2750
-F 0 "U?" H 1942 3215 50  0000 C CNN
-F 1 "10M50SCE144C8G" H 1942 3124 50  0000 C CNN
-F 2 "10M50SCE144:QFP50P2200X2200X165-145N" H 2250 2750 50  0001 C CNN
-F 3 "" H 2250 2750 50  0001 C CNN
-	4    2250 2750
+P 1750 2200
+F 0 "U1" H 1442 2665 50  0000 C CNN
+F 1 "10M50SCE144C8G" H 1442 2574 50  0000 C CNN
+F 2 "10M50SCE144:QFP50P2200X2200X165-145N" H 1750 2200 50  0001 C CNN
+F 3 "" H 1750 2200 50  0001 C CNN
+	4    1750 2200
 	-1   0    0    -1
 $EndComp
 Wire Wire Line
-	2950 2550 3400 2550
+	2450 2000 2900 2000
 Wire Wire Line
-	2950 2650 3400 2650
+	2450 2100 2900 2100
 Wire Wire Line
-	2950 2750 3400 2750
+	2450 2200 2900 2200
 Wire Wire Line
-	2950 2850 3400 2850
+	2450 2300 2900 2300
 Wire Wire Line
-	2950 2950 3400 2950
+	2450 2400 2900 2400
 Wire Wire Line
-	2950 3050 3400 3050
+	2450 2500 2900 2500
 Wire Wire Line
-	2950 3150 3400 3150
+	2450 2600 2900 2600
 Wire Wire Line
-	2950 3250 3400 3250
+	2450 2700 2900 2700
 Wire Wire Line
-	2950 3350 3400 3350
-Text Label 3050 2550 0    50   ~ 0
+	2450 2800 2900 2800
+Text Label 2550 2000 0    50   ~ 0
 DOUT1
-Text Label 3050 2650 0    50   ~ 0
+Text Label 2550 2100 0    50   ~ 0
 DOU2
-Text Label 3050 2750 0    50   ~ 0
+Text Label 2550 2200 0    50   ~ 0
 DOUT3
-Text Label 3050 2850 0    50   ~ 0
+Text Label 2550 2300 0    50   ~ 0
 DOUT4
-Text Label 3050 2950 0    50   ~ 0
+Text Label 2550 2400 0    50   ~ 0
 DOUT5
-Text Label 3050 3050 0    50   ~ 0
+Text Label 2550 2500 0    50   ~ 0
 DOUT6
-Text Label 3050 3150 0    50   ~ 0
+Text Label 2550 2600 0    50   ~ 0
 DOUT7
-Text Label 3050 3250 0    50   ~ 0
+Text Label 2550 2700 0    50   ~ 0
 DOUT8
-Text Label 3050 3350 0    50   ~ 0
+Text Label 2550 2800 0    50   ~ 0
 DOUT9
 $EndSCHEMATC
