File: Serializer.sch (KiCad schematic (older format))
At the start: 40 parts, among them J1 U.FL-R-SMT-110, J2 DNL, U1 DS90UB913ATRTVTQ1, U2 TLV7103318DSER

Commit message: sync
Parts:
- C10, C11, C14, C3, C7: symbol Capacitor:GRM033R71A103KA01D -> Serializer-rescue:GRM033R71A103KA01D-Capacitor
- C12, C16, C17: symbol Capacitor:GRM155R60J106ME15D -> Serializer-rescue:GRM155R60J106ME15D-Capacitor
- C13, C15, C2, C5, C6, C8, C?: symbol Capacitor:GRM033R61A104ME15D -> Serializer-rescue:GRM033R61A104ME15D-Capacitor
- J1: symbol dk_Coaxial-Connectors-RF:U_FL-R-SMT_10_ -> Serializer-rescue:U_FL-R-SMT_10_-dk_Coaxial-Connectors-RF
- U1: symbol SERDES:DS90UB933-Q1 -> Serializer-rescue:DS90UB933-Q1-SERDES
- U?: symbol DS90UB953ATRHBRQ1:DS90UB953ATRHBRQ1 -> Serializer-rescue:DS90UB953ATRHBRQ1-DS90UB953ATRHBRQ1
Changed lines of the file:
@@
 VDDD
 $Comp
-L Capacitor:GRM033R61A104ME15D C2
+L Serializer-rescue:GRM033R61A104ME15D-Capacitor C2
 U 1 1 5FF39341
 P 7350 3300
@@
 	7350 3450 7850 3450
 $Comp
-L Capacitor:GRM033R61A104ME15D C5
+L Serializer-rescue:GRM033R61A104ME15D-Capacitor C5
 U 1 1 5FF5EBAF
 P 7350 4000
@@
 	7350 3850 7850 3850
 $Comp
-L Capacitor:GRM033R61A104ME15D C8
+L Serializer-rescue:GRM033R61A104ME15D-Capacitor C8
 U 1 1 600743E5
 P 7350 1900
@@
 $EndComp
 $Comp
-L Capacitor:GRM155R60J106ME15D C12
+L Serializer-rescue:GRM155R60J106ME15D-Capacitor C12
 U 1 1 60074F7D
 P 6850 2600
@@
 $EndComp
 $Comp
-L Capacitor:GRM033R61A104ME15D C13
+L Serializer-rescue:GRM033R61A104ME15D-Capacitor C13
 U 1 1 60075DB5
 P 7350 2600
@@
 VDDCML
 $Comp
-L Capacitor:GRM033R71A103KA01D C10
+L Serializer-rescue:GRM033R71A103KA01D-Capacitor C10
 U 1 1 60071224
 P 7850 1300
@@
 $EndComp
 $Comp
-L Capacitor:GRM033R61A104ME15D C6
+L Serializer-rescue:GRM033R61A104ME15D-Capacitor C6
 U 1 1 6006E176
 P 7350 1300
@@
 	3750 6650 3900 6650
 $Comp
-L SERDES:DS90UB933-Q1 U1
+L Serializer-rescue:DS90UB933-Q1-SERDES U1
 U 1 1 5FF0C6FA
 P -4150 5500
@@
 	-2150 5000 -1850 5000
 $Comp
-L Capacitor:GRM033R61A104ME15D C15
+L Serializer-rescue:GRM033R61A104ME15D-Capacitor C15
 U 1 1 6012F7F8
 P -2250 5000
@@
 $EndComp
 $Comp
-L Capacitor:GRM033R71A103KA01D C3
+L Serializer-rescue:GRM033R71A103KA01D-Capacitor C3
 U 1 1 5FF73F4B
 P 7850 1900
@@
 $EndComp
 $Comp
-L Capacitor:GRM033R71A103KA01D C7
+L Serializer-rescue:GRM033R71A103KA01D-Capacitor C7
 U 1 1 5FF745CE
 P 7850 2600
@@
 $EndComp
 $Comp
-L Capacitor:GRM033R71A103KA01D C11
+L Serializer-rescue:GRM033R71A103KA01D-Capacitor C11
 U 1 1 5FF74D09
 P 7850 3300
@@
 $EndComp
 $Comp
-L Capacitor:GRM033R71A103KA01D C14
+L Serializer-rescue:GRM033R71A103KA01D-Capacitor C14
 U 1 1 5FF753D1
 P 7850 4000
@@
 $EndComp
 $Comp
-L Capacitor:GRM155R60J106ME15D C16
+L Serializer-rescue:GRM155R60J106ME15D-Capacitor C16
 U 1 1 5FF90C32
 P 4100 5450
@@
 $EndComp
 $Comp
-L Capacitor:GRM155R60J106ME15D C17
+L Serializer-rescue:GRM155R60J106ME15D-Capacitor C17
 U 1 1 5FF9192E
 P 4550 5450
@@
 Breakout pads\n
 $Comp
-L dk_Coaxial-Connectors-RF:U_FL-R-SMT_10_ J1
+L Serializer-rescue:U_FL-R-SMT_10_-dk_Coaxial-Connectors-RF J1
 U 1 1 5FFDACBE
 P 2250 5300
@@
 $EndComp
 $Comp
-L DS90UB953ATRHBRQ1:DS90UB953ATRHBRQ1 U?
+L Serializer-rescue:DS90UB953ATRHBRQ1-DS90UB953ATRHBRQ1 U?
 U 1 1 60437C66
 P 800 800
@@
 	4450 1865 4400 1865
 $Comp
-L Capacitor:GRM033R61A104ME15D C?
+L Serializer-rescue:GRM033R61A104ME15D-Capacitor C?
 U 1 1 6057B91E
 P 4300 1610
