File: Mousecam/FPGA.sch (KiCad schematic (older format))
At the start: 3 parts, among them U1 10M50SCE144C8G

Commit message: sync
Connections:
- net SCK: now reaches U1.51 (BK3_IO_11)
- net MOSI: now reaches U1.52 (BK3_IO_12)
- net MISO: now reaches U1.53 (BK3_IO_13)
- net SS_N: now reaches U1.55 (BK3_IO_14)
Changed lines of the file:
@@
 Wire Wire Line
 	9400 3500 9300 3500
+Wire Wire Line
+	4500 2650 4200 2650
+Wire Wire Line
+	4500 2750 4200 2750
+Wire Wire Line
+	4500 2850 4200 2850
+Wire Wire Line
+	4500 2950 4200 2950
+Text HLabel 4200 2650 0    50   Input ~ 0
+SCK
+Text HLabel 4200 2750 0    50   Input ~ 0
+MOSI
+Text HLabel 4200 2850 0    50   Input ~ 0
+MISO
+Text HLabel 4200 2950 0    50   Input ~ 0
+SS_N
 $EndSCHEMATC
