File: Mousecam/_autosave-Mousecam.sch (KiCad schematic (older format))
At the start: 0 parts

Commit message: sync
Parts:
- added J?: Conn_ARM_JTAG_SWD_10, symbol Connector:Conn_ARM_JTAG_SWD_10
Connections:
- wire segments 0 -> 14
Changed lines of the file:
@@
 $EndDescr
 $Sheet
-S 2950 900  3350 1500
+S 1150 1450 3350 1500
 U 607CBC7A
 F0 "Python480" 50
 F1 "Python480.sch" 50
-F2 "MONITOR0" O L 2950 1050 50
-F3 "TRIGGER0" I L 2950 1200 50
-F4 "RESET_N" I L 2950 1300 50
-F5 "SCK" I L 2950 1450 50
-F6 "MOSI" I L 2950 1550 50
-F7 "MISO" O L 2950 1650 50
-F8 "SS_N" I L 2950 1750 50
-F9 "D9" O R 6300 950 50
-F10 "D8" O R 6300 1050 50
-F11 "D7" O R 6300 1150 50
-F12 "D6" O R 6300 1250 50
-F13 "D5" O R 6300 1350 50
-F14 "D4" O R 6300 1450 50
-F15 "LV" O R 6300 2300 50
-F16 "FV" O R 6300 2200 50
-F17 "PXL_CLK" O R 6300 2100 50
-F18 "D3" O R 6300 1550 50
-F19 "D2" O R 6300 1650 50
-F20 "D1" O R 6300 1750 50
-F21 "D0" O R 6300 1850 50
+F2 "MONITOR0" O L 1150 1600 50
+F3 "TRIGGER0" I L 1150 1750 50
+F4 "RESET_N" I L 1150 1850 50
+F5 "SCK" I R 4500 2550 50
+F6 "MOSI" I R 4500 2750 50
+F7 "MISO" O R 4500 2650 50
+F8 "SS_N" I R 4500 2850 50
+F9 "D9" O R 4500 1500 50
+F10 "D8" O R 4500 1600 50
+F11 "D7" O R 4500 1700 50
+F12 "D6" O R 4500 1800 50
+F13 "D5" O R 4500 1900 50
+F14 "D4" O R 4500 2000 50
+F15 "LV" O L 1150 2750 50
+F16 "FV" O L 1150 2650 50
+F17 "PXL_CLK" O L 1150 2550 50
+F18 "D3" O R 4500 2100 50
+F19 "D2" O R 4500 2200 50
+F20 "D1" O R 4500 2300 50
+F21 "D0" O R 4500 2400 50
 $EndSheet
 $Sheet
-S 2400 3250 2100 2950
+S 1800 3300 2100 2950
 U 607CBDDC
 F0 "Serializer" 50
 F1 "Serializer.sch" 50
-F2 "LV" I L 2400 3400 50
-F3 "FV" I L 2400 3500 50
-F4 "D0" I L 2400 3600 50
-F5 "D1" I L 2400 3700 50
-F6 "D2" I L 2400 3800 50
-F7 "D3" I L 2400 3900 50
-F8 "D4" I L 2400 4000 50
-F9 "D5" I L 2400 4100 50
-F10 "D6" I L 2400 4200 50
-F11 "D7" I L 2400 4300 50
-F12 "D8" I L 2400 4400 50
-F13 "D9" I L 2400 4500 50
-F14 "I2C_SCL" I L 2400 5100 50
-F15 "D10" I L 2400 4600 50
-F16 "D11" I L 2400 4700 50
-F17 "PXL_CLK" I L 2400 4900 50
-F18 "I2C_SDA" I L 2400 5200 50
-F19 "CSI_CLKP" I L 2400 5300 50
-F20 "CSI_CLKN" I L 2400 5400 50
-F21 "CSI_D0P" I L 2400 5500 50
-F22 "CSI_D0N" I L 2400 5600 50
-F23 "CSI_D1P" I L 2400 5700 50
-F24 "CSI_D1N" I L 2400 5800 50
-F25 "CSI_D2P" I L 2400 5900 50
-F26 "CSI_D3P" I L 2400 6000 50
-F27 "CSI_D3N" I L 2400 6100 50
+F2 "LV" I L 1800 3450 50
+F3 "FV" I L 1800 3550 50
+F4 "D0" I L 1800 3650 50
+F5 "D1" I L 1800 3750 50
+F6 "D2" I L 1800 3850 50
+F7 "D3" I L 1800 3950 50
+F8 "D4" I L 1800 4050 50
+F9 "D5" I L 1800 4150 50
+F10 "D6" I L 1800 4250 50
+F11 "D7" I L 1800 4350 50
+F12 "D8" I L 1800 4450 50
+F13 "D9" I L 1800 4550 50
+F14 "I2C_SCL" I L 1800 5150 50
+F15 "D10" I L 1800 4650 50
+F16 "D11" I L 1800 4750 50
+F17 "PXL_CLK" I L 1800 4950 50
+F18 "I2C_SDA" I L 1800 5250 50
+F19 "CSI_CLKP" I L 1800 5350 50
+F20 "CSI_CLKN" I L 1800 5450 50
+F21 "CSI_D0P" I L 1800 5550 50
+F22 "CSI_D0N" I L 1800 5650 50
+F23 "CSI_D1P" I L 1800 5750 50
+F24 "CSI_D1N" I L 1800 5850 50
+F25 "CSI_D2P" I L 1800 5950 50
+F26 "CSI_D3P" I L 1800 6050 50
+F27 "CSI_D3N" I L 1800 6150 50
 $EndSheet
 $Sheet
-S 7500 2200 1800 3050
+S 6000 1250 1800 3050
 U 607CBD48
 F0 "FPGA" 50
 F1 "FPGA.sch" 50
-F2 "JTAGEN" I L 7500 2300 50
-F3 "TMS" I L 7500 2400 50
-F4 "TCK" I L 7500 2500 50
-F5 "TDI" I L 7500 2600 50
-F6 "TDO" I L 7500 2700 50
-F7 "D9" I L 7500 2950 50
-F8 "D8" I L 7500 3050 50
-F9 "D7" I L 7500 3150 50
-F10 "D6" I L 7500 3250 50
-F11 "D5" I L 7500 3350 50
-F12 "D4" I L 7500 3450 50
-F13 "D3" I L 7500 3550 50
-F14 "D2" I L 7500 3650 50
-F15 "D1" I L 7500 3750 50
-F16 "D0" I L 7500 3850 50
-F17 "VCC_ONE" I L 7500 4100 50
-F18 "VCCIO1A" I L 7500 4250 50
-F19 "VCCIO1B" I L 7500 4350 50
-F20 "VCCIO2" I L 7500 4450 50
-F21 "VCCIO4" I L 7500 4650 50
-F22 "VCCIO5" I L 7500 4750 50
-F23 "VCCIO6" I L 7500 4850 50
-F24 "VCCIO7" I L 7500 4950 50
-F25 "VCCIO8" I L 7500 5050 50
-F26 "VCCIO3" I L 7500 4550 50
+F2 "D9" I L 6000 1500 50
+F3 "D8" I L 6000 1600 50
+F4 "D7" I L 6000 1700 50
+F5 "D6" I L 6000 1800 50
+F6 "D5" I L 6000 1900 50
+F7 "D4" I L 6000 2000 50
+F8 "D3" I L 6000 2100 50
+F9 "D2" I L 6000 2200 50
+F10 "D1" I L 6000 2300 50
+F11 "D0" I L 6000 2400 50
+F12 "VCC_ONE" I L 6000 3150 50
+F13 "VCCIO1A" I L 6000 3300 50
+F14 "VCCIO1B" I L 6000 3400 50
+F15 "VCCIO2" I L 6000 3500 50
+F16 "VCCIO4" I L 6000 3700 50
+F17 "VCCIO5" I L 6000 3800 50
+F18 "VCCIO6" I L 6000 3900 50
+F19 "VCCIO7" I L 6000 4000 50
+F20 "VCCIO8" I L 6000 4100 50
+F21 "VCCIO3" I L 6000 3600 50
+F22 "JTAGEN" I R 7800 1400 50
+F23 "TMS" I R 7800 1500 50
+F24 "TCK" I R 7800 1600 50
+F25 "TDI" I R 7800 1700 50
+F26 "TDO" I R 7800 1800 50
+F27 "SCK" I L 6000 2550 50
+F28 "MOSI" I L 6000 2650 50
+F29 "MISO" I L 6000 2750 50
+F30 "SS_N" I L 6000 2850 50
 $EndSheet
+Wire Wire Line
+	4500 1500 6000 1500
+Wire Wire Line
+	4500 1600 6000 1600
+Wire Wire Line
+	4500 1700 6000 1700
+Wire Wire Line
+	4500 1800 6000 1800
+Wire Wire Line
+	4500 1900 6000 1900
+Wire Wire Line
+	4500 2000 6000 2000
+Wire Wire Line
+	4500 2100 6000 2100
+Wire Wire Line
+	4500 2200 6000 2200
+Wire Wire Line
+	4500 2300 6000 2300
+Wire Wire Line
+	4500 2400 6000 2400
+Wire Wire Line
+	4500 2550 6000 2550
+Wire Wire Line
+	4500 2650 6000 2650
+Wire Wire Line
+	4500 2750 6000 2750
+Wire Wire Line
+	4500 2850 6000 2850
+$Comp
+L Connector:Conn_ARM_JTAG_SWD_10 J?
+U 1 1 60806A59
+P 9700 1700
+F 0 "J?" H 9256 1654 50  0000 R CNN
+F 1 "Conn_ARM_JTAG_SWD_10" H 9256 1745 50  0000 R CNN
+F 2 "" H 9700 1700 50  0001 C CNN
+F 3 "http://infocenter.arm.com/help/topic/com.arm.doc.ddi0314h/DDI0314H_coresight_components_trm.pdf" V 9350 450 50  0001 C CNN
+	1    9700 1700
+	-1   0    0    1
+$EndComp
 $EndSCHEMATC
