File: Mousecam/Serializer.sch (KiCad schematic (older format))
At the start: 40 parts, among them J1 U.FL-R-SMT-110, J2 DNL, U1 DS90UB913ATRTVTQ1, U2 TLV7103318DSER

Commit message: sync
Parts:
- renumbered C2 to C?, C21 to C?, C5 to C?, C3 to C?, C7 to C?, C11 to C?, C14 to C?, C4 to C?, C16 to C?, C17 to C?, C9 to C?, C6 to C?, C10 to C?, C8 to C?, C12 to C?, C13 to C?, C15 to C?, C18 to C?, C19 to C?, C20 to C?, C1 to C?, J1 to J?, J2 to J?, J_coax_gnd1 to J_coax_gnd?, L1 to L?, L2 to L?, L3 to L?, L4 to L?, R3 to R?, R6 to R?, R1 to R?, R2 to R?, R4 to R?, R5 to R?, U1 to U?, U2 to U?
Changed lines of the file:
@@
 VDDD
 $Comp
-L Serializer-rescue:GRM033R61A104ME15D-Capacitor C2
+L Serializer-rescue:GRM033R61A104ME15D-Capacitor C?
 U 1 1 5FF39341
 P 7350 3300
@@
 	7350 3450 7850 3450
 $Comp
-L Serializer-rescue:GRM033R61A104ME15D-Capacitor C5
+L Serializer-rescue:GRM033R61A104ME15D-Capacitor C?
 U 1 1 5FF5EBAF
 P 7350 4000
@@
 	7850 3450 7850 3400
 $Comp
-L power:GND #PWR02
+L power:GND #PWR?
 U 1 1 5FF64AA6
 P 7350 4200
@@
 	7350 4150 7350 4100
 $Comp
-L power:+1V8 #PWR05
+L power:+1V8 #PWR?
 U 1 1 5FF697ED
 P 7850 3050
@@
 $EndComp
 $Comp
-L power:+1V8 #PWR04
+L power:+1V8 #PWR?
 U 1 1 5FF6A0B9
 P 7850 3750
@@
 MODE
 $Comp
-L Device:C_Small C4
+L Device:C_Small C?
 U 1 1 5FF87FC9
 P 6850 1900
@@
 Connection ~ 7350 2050
 $Comp
-L power:GND #PWR03
+L power:GND #PWR?
 U 1 1 5FF8D880
 P 7350 2150
@@
 VDDPLL
 $Comp
-L Device:L_Small L1
+L Device:L_Small L?
 U 1 1 5FF90959
 P 8150 1750
@@
 $EndComp
 $Comp
-L power:+1V8 #PWR06
+L power:+1V8 #PWR?
 U 1 1 5FF94686
 P 8350 1700
@@
 	7350 3850 7850 3850
 $Comp
-L Serializer-rescue:GRM033R61A104ME15D-Capacitor C8
+L Serializer-rescue:GRM033R61A104ME15D-Capacitor C?
 U 1 1 600743E5
 P 7350 1900
@@
 $EndComp
 $Comp
-L Serializer-rescue:GRM155R60J106ME15D-Capacitor C12
+L Serializer-rescue:GRM155R60J106ME15D-Capacitor C?
 U 1 1 60074F7D
 P 6850 2600
@@
 $EndComp
 $Comp
-L Serializer-rescue:GRM033R61A104ME15D-Capacitor C13
+L Serializer-rescue:GRM033R61A104ME15D-Capacitor C?
 U 1 1 60075DB5
 P 7350 2600
@@
 $EndComp
 $Comp
-L Device:L_Small L2
+L Device:L_Small L?
 U 1 1 6008139F
 P 8150 2450
@@
 	8350 2450 8350 2350
 $Comp
-L power:+1V8 #PWR010
+L power:+1V8 #PWR?
 U 1 1 6008C0C3
 P 8350 2350
@@
 VDDCML
 $Comp
-L Serializer-rescue:GRM033R71A103KA01D-Capacitor C10
+L Serializer-rescue:GRM033R71A103KA01D-Capacitor C?
 U 1 1 60071224
 P 7850 1300
@@
 $EndComp
 $Comp
-L Serializer-rescue:GRM033R61A104ME15D-Capacitor C6
+L Serializer-rescue:GRM033R61A104ME15D-Capacitor C?
 U 1 1 6006E176
 P 7350 1300
@@
 	7850 1050 7850 1150
 $Comp
-L power:+1V8 #PWR08
+L power:+1V8 #PWR?
 U 1 1 6004EB41
 P 7850 1050
@@
 	6850 1200 6850 1150
 $Comp
-L power:GND #PWR07
+L power:GND #PWR?
 U 1 1 600314E0
 P 7350 1500
@@
 $EndComp
 $Comp
-L Device:C_Small C9
+L Device:C_Small C?
 U 1 1 6002E3A6
 P 6850 1300
@@
 	-2000 5400 -2050 5400
 $Comp
-L power:GND #PWR011
+L power:GND #PWR?
 U 1 1 6015939C
 P -1650 5400
@@
 $EndComp
 $Comp
-L Device:R R1
+L Device:R R?
 U 1 1 601443DA
 P -1850 5400
@@
 	5050 4700 5050 7550
 $Comp
-L Device:L_Small L3
+L Device:L_Small L?
 U 1 1 602E3CB4
 P 3100 5300
@@
 $EndComp
 $Comp
-L Device:L_Small L4
+L Device:L_Small L?
 U 1 1 602E56BF
 P 3550 5300
@@
 $EndComp
 $Comp
-L Device:R_Small_US R2
+L Device:R_Small_US R?
 U 1 1 602E686F
 P 3550 5600
@@
 	4550 5600 4550 5550
 $Comp
-L power:GND #PWR014
+L power:GND #PWR?
 U 1 1 602FE443
 P 4550 5600
@@
 Connection ~ 4550 5600
 $Comp
-L power:+5V #PWR013
+L power:+5V #PWR?
 U 1 1 603454ED
 P 4550 5300
@@
 	2250 6650 2250 6750
 $Comp
-L power:+5V #PWR015
+L power:+5V #PWR?
 U 1 1 603C4B63
 P 1800 6650
@@
 $EndComp
 $Comp
-L Device:C_Small C18
+L Device:C_Small C?
 U 1 1 603CA409
 P 1950 6950
@@
 $EndComp
 $Comp
-L power:GND #PWR021
+L power:GND #PWR?
 U 1 1 60516C41
 P 2350 7300
@@
 Connection ~ 1950 6650
 $Comp
-L Device:R_Small R3
+L Device:R_Small R?
 U 1 1 5FF312E4
 P 5600 1700
@@
 $EndComp
 $Comp
-L power:+1V8 #PWR016
+L power:+1V8 #PWR?
 U 1 1 5FF32F4D
 P 5600 1500
@@
 $EndComp
 $Comp
-L power:GND #PWR022
+L power:GND #PWR?
 U 1 1 5FF34524
 P 5600 2300
@@
 	5600 1900 5600 1800
 $Comp
-L Device:C_Small C21
+L Device:C_Small C?
 U 1 1 5FF4CA15
 P 5600 3550
@@
 	5600 3450 5600 3350
 $Comp
-L power:GND #PWR024
+L power:GND #PWR?
 U 1 1 5FF5387B
 P 5600 3750
@@
 	5600 3750 5600 3650
 $Comp
-L power:+1V8 #PWR023
+L power:+1V8 #PWR?
 U 1 1 5FF5DCD7
 P 5600 2950
@@
 	3600 6550 4550 6550
 $Comp
-L power:+3.3V #PWR018
+L power:+3.3V #PWR?
 U 1 1 60405E6D
 P 4650 6550
@@
 $EndComp
 $Comp
-L power:+1V8 #PWR017
+L power:+1V8 #PWR?
 U 1 1 603E3341
 P 3900 6650
@@
 $EndComp
 $Comp
-L power:GND #PWR020
+L power:GND #PWR?
 U 1 1 603F74F6
 P 4550 7050
@@
 $EndComp
 $Comp
-L Device:C_Small C20
+L Device:C_Small C?
 U 1 1 603F7011
 P 4550 6850
@@
 $EndComp
 $Comp
-L power:GND #PWR019
+L power:GND #PWR?
 U 1 1 603E2D15
 P 3750 7050
@@
 $EndComp
 $Comp
-L Device:C_Small C19
+L Device:C_Small C?
 U 1 1 603D8DB0
 P 3750 6850
@@
 	3750 6650 3900 6650
 $Comp
-L Serializer-rescue:DS90UB933-Q1-SERDES U1
+L Serializer-rescue:DS90UB933-Q1-SERDES U?
 U 1 1 5FF0C6FA
 P -4150 5500
@@
 	5600 3050 5600 2950
 $Comp
-L power:GND #PWR025
+L power:GND #PWR?
 U 1 1 60250FCD
 P -2800 7550
@@
 	-2800 6500 -2500 6500
 $Comp
-L power:GND #PWR026
+L power:GND #PWR?
 U 1 1 6025B9D6
 P -2500 6500
@@
 	7350 3550 7350 3450
 $Comp
-L power:GND #PWR01
+L power:GND #PWR?
 U 1 1 5FF3BD35
 P 7350 3550
@@
 $EndComp
 $Comp
-L power:GND #PWR0101
+L power:GND #PWR?
 U 1 1 6038339E
 P 7350 2850
@@
 	7850 1450 7850 1400
 $Comp
-L Connector_Generic:Conn_01x01 J_coax_gnd1
+L Connector_Generic:Conn_01x01 J_coax_gnd?
 U 1 1 6040543E
 P 1100 5300
@@
 $EndComp
 $Comp
-L power:GND #PWR09
+L power:GND #PWR?
 U 1 1 60407505
 P 1100 5600
@@
 $EndComp
 $Comp
-L power:GND #PWR012
+L power:GND #PWR?
 U 1 1 60411FA3
 P 2250 5600
@@
 	1100 5600 1100 5500
 $Comp
-L Device:R_Small R4
+L Device:R_Small R?
 U 1 1 6046BCC8
 P 5600 2100
@@
 $EndComp
 $Comp
-L Device:R_Small R5
+L Device:R_Small R?
 U 1 1 6046D2B3
 P 5600 3150
@@
 	-2450 5250 -2450 5400
 $Comp
-L Device:C C1
+L Device:C C?
 U 1 1 6047D677
 P -2200 5400
@@
 	-2150 5000 -1850 5000
 $Comp
-L Serializer-rescue:GRM033R61A104ME15D-Capacitor C15
+L Serializer-rescue:GRM033R61A104ME15D-Capacitor C?
 U 1 1 6012F7F8
 P -2250 5000
@@
 $EndComp
 $Comp
-L Serializer-rescue:GRM033R71A103KA01D-Capacitor C3
+L Serializer-rescue:GRM033R71A103KA01D-Capacitor C?
 U 1 1 5FF73F4B
 P 7850 1900
@@
 $EndComp
 $Comp
-L Serializer-rescue:GRM033R71A103KA01D-Capacitor C7
+L Serializer-rescue:GRM033R71A103KA01D-Capacitor C?
 U 1 1 5FF745CE
 P 7850 2600
@@
 $EndComp
 $Comp
-L Serializer-rescue:GRM033R71A103KA01D-Capacitor C11
+L Serializer-rescue:GRM033R71A103KA01D-Capacitor C?
 U 1 1 5FF74D09
 P 7850 3300
@@
 $EndComp
 $Comp
-L Serializer-rescue:GRM033R71A103KA01D-Capacitor C14
+L Serializer-rescue:GRM033R71A103KA01D-Capacitor C?
 U 1 1 5FF753D1
 P 7850 4000
@@
 $EndComp
 $Comp
-L Serializer-rescue:GRM155R60J106ME15D-Capacitor C16
+L Serializer-rescue:GRM155R60J106ME15D-Capacitor C?
 U 1 1 5FF90C32
 P 4100 5450
@@
 $EndComp
 $Comp
-L Serializer-rescue:GRM155R60J106ME15D-Capacitor C17
+L Serializer-rescue:GRM155R60J106ME15D-Capacitor C?
 U 1 1 5FF9192E
 P 4550 5450
@@
 $EndComp
 $Comp
-L Serializer-rescue:TLV7103318DSER-TLV7103318DSER U2
+L Serializer-rescue:TLV7103318DSER-TLV7103318DSER U?
 U 1 1 603AD9B0
 P 2300 6550
@@
 Breakout pads\n
 $Comp
-L Serializer-rescue:U_FL-R-SMT_10_-dk_Coaxial-Connectors-RF J1
+L Serializer-rescue:U_FL-R-SMT_10_-dk_Coaxial-Connectors-RF J?
 U 1 1 5FFDACBE
 P 2250 5300
@@
 $EndComp
 $Comp
-L power:GND #PWR0102
+L power:GND #PWR?
 U 1 1 60016AE8
 P 6100 5450
@@
 	6100 5450 5900 5450
 $Comp
-L power:+5V #PWR0103
+L power:+5V #PWR?
 U 1 1 6001D50C
 P 6100 5550
@@
 D11
 $Comp
-L Device:R_Small_US R6
+L Device:R_Small_US R?
 U 1 1 601021F6
 P 3050 5600
@@
 	2800 5300 3000 5300
 $Comp
-L Connector_Generic:Conn_01x05 J2
+L Connector_Generic:Conn_01x05 J?
 U 1 1 5FFF727F
 P 5700 5450

Commit message: sync
Parts:
- removed C?: 1uF, symbol Device:C_Small
- removed C? (x2): 1uF, Capacitor_SMD:C_0201_0603Metric, symbol Device:C_Small
- removed U?: TLV7103318DSER, DSE6, symbol Serializer-rescue:TLV7103318DSER-TLV7103318DSER
Other:
- note removed: "Low-dropout (LDO)\nLinear Voltage Regulator\n"
Changed lines of the file:
@@
 Text Notes 700  5050 0    98   ~ 0
 Power over coax \n\n
-Wire Notes Line
-	650  4700 5050 4700
-Wire Notes Line
-	650  7550 5050 7550
-Wire Notes Line
-	650  4700 650  7550
-Wire Notes Line
-	5050 4700 5050 7550
 $Comp
 L Device:L_Small L?
@@
 $EndComp
 Connection ~ 4550 5300
-Wire Notes Line
-	5050 5950 600  5950
 Connection ~ 4100 5300
 Wire Wire Line
@@
 Text Label 4720 1610 2    39   ~ 0
 DOUT_P
-$Comp
-L Serializer-rescue:TLV7103318DSER-TLV7103318DSER U?
-U 1 1 603AD9B0
-P 2300 6550
-F 0 "U?" H 2950 6900 60  0000 C CNN
-F 1 "TLV7103318DSER" H 3000 6800 60  0000 C CNN
-F 2 "DSE6" H 3400 6790 60  0001 C CNN
-F 3 "" H 2300 6550 60  0000 C CNN
-	1    2300 6550
-	1    0    0    -1
-$EndComp
-Wire Wire Line
-	3750 6650 3900 6650
-Wire Wire Line
-	3750 6750 3750 6650
-Connection ~ 3750 6650
-Wire Wire Line
-	3600 6650 3750 6650
-$Comp
-L Device:C_Small C?
-U 1 1 603D8DB0
-P 3750 6850
-F 0 "C?" H 3842 6896 50  0000 L CNN
-F 1 "1uF" H 3842 6805 50  0000 L CNN
-F 2 "Capacitor_SMD:C_0201_0603Metric" H 3750 6850 50  0001 C CNN
-F 3 "~" H 3750 6850 50  0001 C CNN
-	1    3750 6850
-	1    0    0    -1
-$EndComp
-$Comp
-L power:GND #PWR?
-U 1 1 603E2D15
-P 3750 7050
-F 0 "#PWR?" H 3750 6800 50  0001 C CNN
-F 1 "GND" H 3755 6877 50  0000 C CNN
-F 2 "" H 3750 7050 50  0001 C CNN
-F 3 "" H 3750 7050 50  0001 C CNN
-	1    3750 7050
-	1    0    0    -1
-$EndComp
-$Comp
-L Device:C_Small C?
-U 1 1 603F7011
-P 4550 6850
-F 0 "C?" H 4642 6896 50  0000 L CNN
-F 1 "1uF" H 4642 6805 50  0000 L CNN
-F 2 "Capacitor_SMD:C_0201_0603Metric" H 4550 6850 50  0001 C CNN
-F 3 "~" H 4550 6850 50  0001 C CNN
-	1    4550 6850
-	1    0    0    -1
-$EndComp
-$Comp
-L power:GND #PWR?
-U 1 1 603F74F6
-P 4550 7050
-F 0 "#PWR?" H 4550 6800 50  0001 C CNN
-F 1 "GND" H 4555 6877 50  0000 C CNN
-F 2 "" H 4550 7050 50  0001 C CNN
-F 3 "" H 4550 7050 50  0001 C CNN
-	1    4550 7050
-	1    0    0    -1
-$EndComp
-$Comp
-L power:+1V8 #PWR?
-U 1 1 603E3341
-P 3900 6650
-F 0 "#PWR?" H 3900 6500 50  0001 C CNN
-F 1 "+1V8" V 3915 6778 50  0000 L CNN
-F 2 "" H 3900 6650 50  0001 C CNN
-F 3 "" H 3900 6650 50  0001 C CNN
-	1    3900 6650
-	0    1    1    0
-$EndComp
-$Comp
-L power:+3.3V #PWR?
-U 1 1 60405E6D
-P 4650 6550
-F 0 "#PWR?" H 4650 6400 50  0001 C CNN
-F 1 "+3.3V" V 4665 6678 50  0000 L CNN
-F 2 "" H 4650 6550 50  0001 C CNN
-F 3 "" H 4650 6550 50  0001 C CNN
-	1    4650 6550
-	0    1    1    0
-$EndComp
-Wire Wire Line
-	3600 6550 4550 6550
-Wire Wire Line
-	4550 6550 4550 6750
-Connection ~ 4550 6550
-Wire Wire Line
-	4550 6550 4650 6550
-Wire Wire Line
-	3750 7050 3750 6950
-Wire Wire Line
-	4550 7050 4550 6950
-Wire Wire Line
-	2950 7250 2950 7300
-Wire Wire Line
-	1800 6650 1950 6650
-Wire Wire Line
-	1950 6650 2250 6650
-Connection ~ 1950 6650
-Wire Wire Line
-	1950 6850 1950 6650
-Wire Wire Line
-	1950 7300 1950 7050
-Wire Wire Line
-	2950 7300 2350 7300
-Wire Wire Line
-	1950 7300 2350 7300
-Connection ~ 2350 7300
-$Comp
-L power:GND #PWR?
-U 1 1 60516C41
-P 2350 7300
-F 0 "#PWR?" H 2350 7050 50  0001 C CNN
-F 1 "GND" H 2355 7127 50  0000 C CNN
-F 2 "" H 2350 7300 50  0001 C CNN
-F 3 "" H 2350 7300 50  0001 C CNN
-	1    2350 7300
-	1    0    0    -1
-$EndComp
-$Comp
-L Device:C_Small C?
-U 1 1 603CA409
-P 1950 6950
-F 0 "C?" H 2042 6996 50  0000 L CNN
-F 1 "1uF" H 2042 6905 50  0000 L CNN
-F 2 "" H 1950 6950 50  0001 C CNN
-F 3 "~" H 1950 6950 50  0001 C CNN
-	1    1950 6950
-	1    0    0    -1
-$EndComp
-$Comp
-L power:+5V #PWR?
-U 1 1 603C4B63
-P 1800 6650
-F 0 "#PWR?" H 1800 6500 50  0001 C CNN
-F 1 "+5V" V 1815 6778 50  0000 L CNN
-F 2 "" H 1800 6650 50  0001 C CNN
-F 3 "" H 1800 6650 50  0001 C CNN
-	1    1800 6650
-	0    -1   -1   0
-$EndComp
-Wire Wire Line
-	2250 6650 2250 6750
-Connection ~ 2250 6650
-Wire Wire Line
-	2300 6650 2250 6650
-Wire Wire Line
-	2250 6750 2300 6750
-Wire Wire Line
-	2250 6550 2250 6650
-Wire Wire Line
-	2250 6550 2300 6550
-Text Notes 650  6300 0    98   ~ 0
-Low-dropout (LDO)\nLinear Voltage Regulator\n
+Wire Notes Line
+	600  4650 4950 4650
+Wire Notes Line
+	4950 4650 4950 5900
+Wire Notes Line
+	4950 5900 600  5900
+Wire Notes Line
+	600  5900 600  4650
 $EndSCHEMATC
