File: Mousecam_Kicad/sch/FPGA.sch (KiCad schematic (older format))
At the start: 3 parts

Commit message: updated relative path for libs
Parts:
- removed U? (x3): 10M50SCE144C8G, 10M50SCE144:QFP50P2200X2200X165-145N, symbol Mousecam-rescue:10M50SCE144C8G-10M50SCE
- added U6: 10M50SCE144C8G, 10M50SCE144:QFP50P2200X2200X165-145N, symbol 10M50SCE:10M50SCE144C8G
Changed lines of the file:
@@
 Comment4 ""
 $EndDescr
-$Comp
-L Mousecam-rescue:10M50SCE144C8G-10M50SCE U?
-U 2 1 6083533B
-P 7150 1950
-F 0 "U?" H 7278 1696 50  0000 L CNN
-F 1 "10M50SCE144C8G" H 7278 1605 50  0000 L CNN
-F 2 "10M50SCE144:QFP50P2200X2200X165-145N" H 6600 2250 50  0001 C CNN
-F 3 "" H 7150 1950 50  0001 C CNN
-	2    7150 1950
-	1    0    0    -1
-$EndComp
-$Comp
-L Mousecam-rescue:10M50SCE144C8G-10M50SCE U?
-U 10 1 60851983
-P 9900 4350
-F 0 "U?" H 9917 1385 50  0000 C CNN
-F 1 "10M50SCE144C8G" H 9917 1476 50  0000 C CNN
-F 2 "10M50SCE144:QFP50P2200X2200X165-145N" H 9350 6200 50  0001 C CNN
-F 3 "" H 9900 5450 50  0001 C CNN
-	10   9900 4350
-	1    0    0    1
-$EndComp
 Wire Wire Line
 	9400 1750 9250 1750
@@
 	9250 1850 9250 1950
 $Comp
-L power:GND #PWR?
+L power:GND #PWR032
 U 1 1 60867786
 P 9200 6200
-F 0 "#PWR?" H 9200 5950 50  0001 C CNN
+F 0 "#PWR032" H 9200 5950 50  0001 C CNN
 F 1 "GND" V 9205 6072 50  0000 R CNN
 F 2 "" H 9200 6200 50  0001 C CNN
@@
 SS_N
 $Comp
-L Mousecam-rescue:10M50SCE144C8G-10M50SCE U?
-U 4 1 6082CFF3
+L 10M50SCE:10M50SCE144C8G U6
+U 10 1 608C607E
+P 9900 4350
+F 0 "U6" H 9917 1385 50  0000 C CNN
+F 1 "10M50SCE144C8G" H 9917 1476 50  0000 C CNN
+F 2 "10M50SCE144:QFP50P2200X2200X165-145N" H 9350 6200 50  0001 C CNN
+F 3 "" H 9900 5450 50  0001 C CNN
+	10   9900 4350
+	1    0    0    1
+$EndComp
+$Comp
+L 10M50SCE:10M50SCE144C8G U6
+U 2 1 608EEFD0
+P 7150 1950
+F 0 "U6" H 7278 1696 50  0000 L CNN
+F 1 "10M50SCE144C8G" H 7278 1605 50  0000 L CNN
+F 2 "10M50SCE144:QFP50P2200X2200X165-145N" H 6600 3800 50  0001 C CNN
+F 3 "" H 7150 3050 50  0001 C CNN
+	2    7150 1950
+	1    0    0    -1
+$EndComp
+$Comp
+L 10M50SCE:10M50SCE144C8G U6
+U 4 1 609009F4
 P 5200 1850
-F 0 "U?" H 5328 1446 50  0000 L CNN
+F 0 "U6" H 5328 1446 50  0000 L CNN
 F 1 "10M50SCE144C8G" H 5328 1355 50  0000 L CNN
 F 2 "10M50SCE144:QFP50P2200X2200X165-145N" H 4650 3700 50  0001 C CNN

Commit message: updated relative path for libs
Parts:
- U6: footprint 10M50SCE144:QFP50P2200X2200X165-145N -> 10m50sce:QFP50P2200X2200X165_145N
Changed lines of the file:
@@
 F 0 "U6" H 9917 1385 50  0000 C CNN
 F 1 "10M50SCE144C8G" H 9917 1476 50  0000 C CNN
-F 2 "10M50SCE144:QFP50P2200X2200X165-145N" H 9350 6200 50  0001 C CNN
+F 2 "10m50sce:QFP50P2200X2200X165_145N" H 9350 6200 50  0001 C CNN
 F 3 "" H 9900 5450 50  0001 C CNN
 	10   9900 4350
@@
 F 0 "U6" H 7278 1696 50  0000 L CNN
 F 1 "10M50SCE144C8G" H 7278 1605 50  0000 L CNN
-F 2 "10M50SCE144:QFP50P2200X2200X165-145N" H 6600 3800 50  0001 C CNN
+F 2 "10m50sce:QFP50P2200X2200X165_145N" H 6600 3800 50  0001 C CNN
 F 3 "" H 7150 3050 50  0001 C CNN
 	2    7150 1950
@@
 F 0 "U6" H 5328 1446 50  0000 L CNN
 F 1 "10M50SCE144C8G" H 5328 1355 50  0000 L CNN
-F 2 "10M50SCE144:QFP50P2200X2200X165-145N" H 4650 3700 50  0001 C CNN
+F 2 "10m50sce:QFP50P2200X2200X165_145N" H 4650 3700 50  0001 C CNN
 F 3 "" H 5200 2950 50  0001 C CNN
 	4    5200 1850
