File: Mousecam_Kicad/sch/Python480.sch (KiCad schematic (older format))
At the start: 29 parts, among them U1 NOIP1SN0480A, U2 LM321, U3 NCP163AMX330TBG, X1 SG-210STF

Commit message: sync
Parts:
- removed C1, C10, C11, C12, C15, C16, C17, C19, C2, C3, C4, C5, C6, C7, C8, C9: GRM033R61A104ME15D, Capacitor_SMD:C_0603_1608Metric_Pad1.05x0.95mm_HandSolder, symbol Python480-rescue:GRM033R61A104ME15D-Capacitor
- removed U1: NOIP1SN0480A, .Package_BGA:BGA88CP50_8X11_493X613X75B25, symbol Python480-rescue:NOIP1SN0480A-Image_Sensor
- added C? (x16): 0.1uF, symbol Device:C_Small
- added U?: NOIP1SN0480A-Image_Sensor, .Package_BGA:BGA88CP50_8X11_493X613X75B25, symbol Python480_rescue:NOIP1SN0480A-Image_Sensor
Connections:
- wire segments 113 -> 97

Commit message: updated relative path for libs
Parts:
- removed C13, C14, C18, C20, C21: GRM033R61A104ME15D, Capacitor_SMD:C_0603_1608Metric_Pad1.05x0.95mm_HandSolder, symbol Python480-rescue:GRM033R61A104ME15D-Capacitor
- removed L2: BLM18AG601SN1D, IND_BLM18_0603_MUR, symbol Python480-rescue:BLM18AG601SN1D-BLM18AG601SN1D
- removed R1: ERJ-1GEF1022C, Resistor_SMD:R_0603_1608Metric_Pad1.05x0.95mm_HandSolder, symbol Python480-rescue:ERJ-1GEF1022C-Resistor
- removed U3: NCP163AMX330TBG, .Package_QFN:UQFN_MCP1711, symbol Python480-rescue:MCP1711-doragasu
- added C22, C23: 10uF, Capacitor_SMD:C_0603_1608Metric_Pad1.05x0.95mm_HandSolder, symbol Device:C_Small
- added C25: 4.7uF, Capacitor_SMD:C_0603_1608Metric_Pad1.05x0.95mm_HandSolder, symbol Device:C_Small
- added C26, C28: 1uF, Capacitor_SMD:C_0603_1608Metric_Pad1.05x0.95mm_HandSolder, symbol Device:C_Small
- added R5: 47.7 kOhm, symbol Device:R_Small
- added U4: BLM18AG601SN1D, symbol BLM18AG601SN1D:BLM18AG601SN1D
- added U5: NCP163AMX180TBG, XDFN4_711AJ_ONS, symbol NCP163AMX180TBG:NCP163AMX180TBG
- C10, C11, C12, C13, C14, C15, C16, C17, C18, C19, C20, C21, C24, C27, C8, C9: renamed from C?; footprint (none) -> Capacitor_SMD:C_0603_1608Metric_Pad1.05x0.95mm_HandSolder
- U3: renamed from U?; symbol Python480_rescue:NOIP1SN0480A-Image_Sensor -> NOIP1SN0480A-STI1:NOIP1SN0480A-STI1
Connections:
- wire segments 97 -> 99

Commit message: updated relative path for libs
Parts:
- removed C27: 0.1uF, Capacitor_SMD:C_0603_1608Metric_Pad1.05x0.95mm_HandSolder, symbol Device:C_Small
- removed L1: BLM18AG601SN1D, IND_BLM18_0603_MUR, symbol Python480-rescue:BLM18AG601SN1D-BLM18AG601SN1D
- removed R2: DNL, Resistor_SMD:R_0603_1608Metric_Pad1.05x0.95mm_HandSolder, symbol Device:R_Small_US
- removed X1: SG-210STF, Oscillator:Oscillator_SMD_SeikoEpson_SG210-4Pin_2.5x2.0mm, symbol Oscillator:SG-210STF
- added U9: BLM18AG601SN1D, BLM18AG601SN1D:BLM18AG601SN1D, symbol BLM18AG601SN1D:BLM18AG601SN1D
- R5: footprint (none) -> Resistor_SMD:R_0603_1608Metric_Pad1.05x0.95mm_HandSolder
- U3: footprint .Package_BGA:BGA88CP50_8X11_493X613X75B25 -> (none)
- U4: footprint (none) -> BLM18AG601SN1D:BLM18AG601SN1D
- U5: footprint XDFN4_711AJ_ONS -> NCP163AMX180TBG:NCP163AMX180TBG
Connections:
- wire segments 99 -> 93
Other:
- note removed: "Oscillator"
Changed lines of the file:
@@
 Wire Notes Line
 	500  500  500  5950
-Wire Notes Line
-	8350 2200 10750 2200
-Wire Notes Line
-	10750 2200 10750 500
-Wire Notes Line
-	10750 500  8350 500
-Wire Notes Line
-	8350 500  8350 2200
 Wire Wire Line
 	4500 2200 5050 2200
@@
 Wire Wire Line
 	6850 4900 7450 4900
-$Comp
-L Python480-rescue:BLM18AG601SN1D-BLM18AG601SN1D L1
-U 1 1 603FF823
-P 5050 2200
-F 0 "L1" H 5350 2529 60  0000 C CNN
-F 1 "BLM18AG601SN1D" H 5350 2423 60  0000 C CNN
-F 2 "IND_BLM18_0603_MUR" H 5325 1915 60  0001 C CNN
-F 3 "https://www.murata.com/en-us/products/productdata/8796738650142/ENFA0003.pdf" H 5050 2200 60  0001 C CNN
-F 4 "600 Ohms @ 100MHz" H 5350 2325 50  0000 C CNN "Note"
-	1    5050 2200
-	1    0    0    -1
-$EndComp
-$Comp
-L Oscillator:SG-210STF X1
-U 1 1 6039666F
-P 9450 1500
-F 0 "X1" H 9650 1150 50  0000 L CNN
-F 1 "SG-210STF" H 9500 1250 50  0000 L CNN
-F 2 "Oscillator:Oscillator_SMD_SeikoEpson_SG210-4Pin_2.5x2.0mm" H 9900 1150 50  0001 C CNN
-F 3 "https://support.epson.biz/td/api/doc_check.php?mode=dl&lang=en&Parts=SG-210STF" H 9350 1500 50  0001 C CNN
-	1    9450 1500
-	1    0    0    -1
-$EndComp
-$Comp
-L power:+3V3 #PWR018
-U 1 1 6039760F
-P 8450 1500
-F 0 "#PWR018" H 8450 1350 50  0001 C CNN
-F 1 "+3V3" H 8465 1673 50  0000 C CNN
-F 2 "" H 8450 1500 50  0001 C CNN
-F 3 "" H 8450 1500 50  0001 C CNN
-	1    8450 1500
-	1    0    0    -1
-$EndComp
-$Comp
-L Device:R_Small_US R2
-U 1 1 6039AAE7
-P 8850 1500
-F 0 "R2" V 8645 1500 50  0000 C CNN
-F 1 "DNL" V 8736 1500 50  0000 C CNN
-F 2 "Resistor_SMD:R_0603_1608Metric_Pad1.05x0.95mm_HandSolder" H 8850 1500 50  0001 C CNN
-F 3 "~" H 8850 1500 50  0001 C CNN
-	1    8850 1500
-	0    1    1    0
-$EndComp
-Wire Wire Line
-	9150 1500 8950 1500
-Wire Wire Line
-	8750 1500 8450 1500
-$Comp
-L power:GND #PWR019
-U 1 1 603A7E17
-P 9450 1800
-F 0 "#PWR019" H 9450 1550 50  0001 C CNN
-F 1 "GND" H 9455 1627 50  0000 C CNN
-F 2 "" H 9450 1800 50  0001 C CNN
-F 3 "" H 9450 1800 50  0001 C CNN
-	1    9450 1800
-	1    0    0    -1
-$EndComp
-Wire Wire Line
-	9750 1500 10100 1500
-Text Label 10100 1500 2    50   ~ 0
-CLK_PLL
-$Comp
-L power:GND #PWR021
-U 1 1 603BCC41
-P 10300 1150
-F 0 "#PWR021" H 10300 900 50  0001 C CNN
-F 1 "GND" V 10305 1022 50  0000 R CNN
-F 2 "" H 10300 1150 50  0001 C CNN
-F 3 "" H 10300 1150 50  0001 C CNN
-	1    10300 1150
-	1    0    0    -1
-$EndComp
-Text Notes 8400 700  0    100  ~ 0
-Oscillator
-$Comp
-L power:+3V3 #PWR020
-U 1 1 603C0811
-P 10300 800
-F 0 "#PWR020" H 10300 650 50  0001 C CNN
-F 1 "+3V3" H 10315 973 50  0000 C CNN
-F 2 "" H 10300 800 50  0001 C CNN
-F 3 "" H 10300 800 50  0001 C CNN
-	1    10300 800
-	1    0    0    -1
-$EndComp
-Wire Wire Line
-	9450 800  9450 1200
-Wire Wire Line
-	9450 800  10300 800
-Wire Wire Line
-	10300 950  10300 800
-Connection ~ 10300 800
 Wire Notes Line
 	8000 4100 11000 4100
@@
 F 0 "U3" H 2625 6281 50  0000 C CNN
 F 1 "NOIP1SN0480A-Image_Sensor" H 2625 6190 50  0000 C CNN
-F 2 ".Package_BGA:BGA88CP50_8X11_493X613X75B25" H 2450 6500 50  0001 C CNN
+F 2 "" H 2450 6500 50  0001 C CNN
 F 3 "" H 2300 6150 50  0001 C CNN
 	1    2550 4100
@@
 	1    0    0    -1
 $EndComp
-$Comp
-L Device:C_Small C?
-U 1 1 60B9B4D6
-P 10300 1050
-AR Path="/607CBDDC/60B9B4D6" Ref="C?"  Part="1"
-AR Path="/607CBC7A/60B9B4D6" Ref="C27"  Part="1"
-F 0 "C27" H 10392 1096 50  0000 L CNN
-F 1 "0.1uF" H 10392 1005 50  0000 L CNN
-F 2 "Capacitor_SMD:C_0603_1608Metric_Pad1.05x0.95mm_HandSolder" H 10300 1050 50  0001 C CNN
-F 3 "~" H 10300 1050 50  0001 C CNN
-	1    10300 1050
-	1    0    0    -1
-$EndComp
 Connection ~ 4950 1400
 Connection ~ 7200 1600
@@
 F 0 "U4" H 6550 5135 50  0000 C CNN
 F 1 "BLM18AG601SN1D" H 6550 5044 50  0000 C CNN
-F 2 "" H 6550 5000 50  0001 C CNN
+F 2 "BLM18AG601SN1D:BLM18AG601SN1D" H 6550 5000 50  0001 C CNN
 F 3 "" H 6550 5000 50  0001 C CNN
 F 4 "600 Ohms @ 100MHz" H 6550 4900 50  0001 C CNN "Spec"
@@
 F 0 "R5" H 1209 5196 50  0000 L CNN
 F 1 "47.7 kOhm" H 1209 5105 50  0000 L CNN
-F 2 "" H 1150 5150 50  0001 C CNN
+F 2 "Resistor_SMD:R_0603_1608Metric_Pad1.05x0.95mm_HandSolder" H 1150 5150 50  0001 C CNN
 F 3 "~" H 1150 5150 50  0001 C CNN
 	1    1150 5150
@@
 F 0 "U5" H 9800 3537 60  0000 C CNN
 F 1 "NCP163AMX180TBG" H 9800 3431 60  0000 C CNN
-F 2 "XDFN4_711AJ_ONS" H 9800 3390 60  0001 C CNN
+F 2 "NCP163AMX180TBG:NCP163AMX180TBG" H 9800 3390 60  0001 C CNN
 F 3 "" H 9000 3150 60  0000 C CNN
 	1    9000 3150
@@
 Wire Wire Line
 	10700 3600 10700 3850
+$Comp
+L BLM18AG601SN1D:BLM18AG601SN1D U9
+U 1 1 608DFB5F
+P 5350 2200
+F 0 "U9" H 5350 2435 50  0000 C CNN
+F 1 "BLM18AG601SN1D" H 5350 2344 50  0000 C CNN
+F 2 "BLM18AG601SN1D:BLM18AG601SN1D" H 5350 2300 50  0001 C CNN
+F 3 "" H 5350 2300 50  0001 C CNN
+	1    5350 2200
+	1    0    0    -1
+$EndComp
 $EndSCHEMATC
